Commit message: Add Collision Tags in the URDF

File: src/my_robot_description/urdf/mobile_base.xacro (robot description, xacro)
@@ -15,11 +15,17 @@
             <origin xyz="0 0 ${base_height / 2}" rpy="0 0 0" />
             <material name="blue" />
-            <xacro:box_inertia m="5.0"
-                               l="${base_length}"
-                               w="${base_width}"
-                               h="${base_height}"
-                               xyz="0 0 ${base_height / 2}"
-                               rpy="0 0 0"/>
         </visual>
+        <collision>
+            <geometry>
+                <box size="${base_length} ${base_width} ${base_height}" />
+            </geometry>
+            <origin xyz="0 0 ${base_height / 2}" rpy="0 0 0" />
+        </collision>
+        <xacro:box_inertia  m="5.0"
+                            l="${base_length}"
+                            w="${base_width}"
+                            h="${base_height}"
+                            xyz="0 0 ${base_height / 2}"
+                            rpy="0 0 0"/>
     </link>
     <xacro:macro name="wheel_link" params="prefix">
@@ -32,4 +38,10 @@
                 <material name="grey" />
             </visual>
+            <collision>
+                <geometry>
+                    <cylinder radius="${wheel_radius}" length="${wheel_length}" />
+                </geometry>
+                <origin xyz="0 0 0" rpy="${pi / 2.0} 0 0" />
+            </collision>
             <xacro:solid_cylinder_inertia m="1.0"
                                           r="${wheel_radius}"
@@ -48,9 +60,15 @@
             <origin xyz="0 0 0" rpy="0 0 0" />
             <material name="grey" />
-            <xacro:solid_sphere_inertia   m="0.5"
-                                          r="${caster_wheel_radius}"
-                                          xyz="0 0 0"
-                                          rpy="0 0 0"/>
         </visual>
+        <collision>
+            <geometry>
+                <sphere radius="${caster_wheel_radius}" />
+            </geometry>
+            <origin xyz="0 0 0" rpy="0 0 0" />
+        </collision>
+        <xacro:solid_sphere_inertia     m="0.5"
+                                        r="${caster_wheel_radius}"
+                                        xyz="0 0 0"
+                                        rpy="0 0 0"/>
     </link>
     <joint name="base_left_wheel_joint" type="continuous">
