Commit message: Add Inertia Tags in the URDF

File: src/my_robot_description/urdf/common_properties.xacro (robot description, xacro)
@@ -7,3 +7,30 @@
         <color rgba="0.5 0.5 0.5 1" />
     </material>
+    <xacro:macro name="box_inertia" params="m l w h xyz rpy">
+        <inertial>
+            <origin xyz="${xyz}" rpy="${rpy}" />
+            <mass value="${m}" />
+            <inertia ixx="${(m/12) * (h*h + l*l)}" ixy="0" ixz="0"
+                     iyy="${(m/12) * (w*w + l*l)}" iyz="0"
+                     izz="${(m/12) * (w*w + h*h)}" />
+        </inertial>
+    </xacro:macro>
+    <xacro:macro name="solid_cylinder_inertia" params="m r h xyz rpy">
+        <inertial>
+            <origin xyz="${xyz}" rpy="${rpy}" />
+            <mass value="${m}" />
+            <inertia ixx="${(m/12) * (3*r*r + h*h)}" ixy="0" ixz="0"
+                     iyy="${(m/12) * (3*r*r + h*h)}" iyz="0"
+                     izz="${(m/2) * (r*r)}" />
+        </inertial>
+    </xacro:macro>
+    <xacro:macro name="solid_sphere_inertia" params="m r xyz rpy">
+        <inertial>
+            <origin xyz="${xyz}" rpy="${rpy}" />
+            <mass value="${m}" />
+            <inertia ixx="${(2/5) * m * r * r}" ixy="0" ixz="0"
+                     iyy="${(2/5) * m * r * r}" iyz="0"
+                     izz="${(2/5) * m * r * r}" />
+        </inertial>
+    </xacro:macro>
 </robot>

File: src/my_robot_description/urdf/mobile_base.xacro (robot description, xacro)
@@ -15,4 +15,10 @@
             <origin xyz="0 0 ${base_height / 2}" rpy="0 0 0" />
             <material name="blue" />
+            <xacro:box_inertia m="5.0"
+                               l="${base_length}"
+                               w="${base_width}"
+                               h="${base_height}"
+                               xyz="0 0 ${base_height / 2}"
+                               rpy="0 0 0"/>
         </visual>
     </link>
@@ -26,4 +32,9 @@
                 <material name="grey" />
             </visual>
+            <xacro:solid_cylinder_inertia m="1.0"
+                                          r="${wheel_radius}"
+                                          h="${wheel_length}"
+                                          xyz="0 0 0"
+                                          rpy="${pi / 2.0} 0 0"/>
         </link>
     </xacro:macro>
@@ -37,4 +48,8 @@
             <origin xyz="0 0 0" rpy="0 0 0" />
             <material name="grey" />
+            <xacro:solid_sphere_inertia   m="0.5"
+                                          r="${caster_wheel_radius}"
+                                          xyz="0 0 0"
+                                          rpy="0 0 0"/>
         </visual>
     </link>

Commit message: Combine RoboticArm With MobileRobot

File: src/my_robot_description/urdf/common_properties.xacro (robot description, xacro)
@@ -6,4 +6,10 @@
     <material name="grey">
         <color rgba="0.5 0.5 0.5 1" />
+    </material>
+    <material name="orange">
+        <color rgba="1 0.5 0 1" />
+    </material>
+    <material name="yellow">
+        <color rgba="1 1 0 1" />
     </material>
     <xacro:macro name="box_inertia" params="m l w h xyz rpy">

File: src/my_robot_description/urdf/my_robot.urdf.xacro (robot description, xacro)
@@ -4,3 +4,11 @@
     <xacro:include filename="mobile_base.xacro" />
     <xacro:include filename="mobile_base_gazebo.xacro" />
+    <xacro:include filename="arm.xacro" />
+    <xacro:include filename="arm_gazebo.xacro" />
+    <joint name="mobile_base_arm_joint" type="fixed">
+        <parent link="base_link"/>
+        <child link="arm_base_link" />
+        <origin xyz="${base_length/4} 0 ${base_height}" rpy="0 0 0" />
+    </joint>
+    <xacro:include filename="camera.xacro" />
 </robot>
